File: audio-breakout.kicad_pcb (KiCad board)
At the start: 2 copper layers, 21.4 x 34 mm, 28 parts, among them IC1 ES8311, J1 AudioJack3, J2 AudioJack3, J3 Conn_01x06_Pin, J4 Conn_01x06_Pin

Commit message: pcb done !!
Parts:
- C1, C10, C11, C12, C13, C14, C15, C16, C17, C2, C3, C4, C5, C6, C7, C8, C9: footprint Capacitor_SMD:C_0201_0603Metric_Pad0.64x0.40mm_HandSolder -> Capacitor_SMD:C_0402_1005Metric
- R1, R2, R3, R4, R5, R6: footprint Resistor_SMD:R_0201_0603Metric_Pad0.64x0.40mm_HandSolder -> Resistor_SMD:R_0402_1005Metric
- moved R3 1.01 mm to (156.3, 51.1)
- moved R1 0.97 mm to (150.5, 45.9)
- moved C11 0.85 mm to (155.3, 50.7)
- moved C4 0.78 mm to (155.8, 46.0)
- moved R5 0.40 mm to (149.9, 51.1)
- moved C9 0.23 mm to (147.4, 47.5)
- moved C16 0.20 mm to (149.9, 50.1)
- moved C15 0.20 mm to (158.9, 42.4)
- moved C10 0.18 mm to (147.4, 50.0)
- moved C1 0.16 mm to (158.9, 44.9)
Routing:
- net GNDA: track 67.0 -> 74.9 mm, vias 6 -> 17
- net +3V3: track 28.6 -> 32.1 mm
- net /I2C_MCLK: track 29.1 -> 27.9 mm
- net Net-(IC1-CE): track 0.79 -> 1.80 mm
- net Net-(IC1-AVDD): track 1.71 -> 2.52 mm
- net Net-(IC1-VMID): track 0.86 -> 1.58 mm
- net /I2C_DSDIN: track 14.0 -> 14.7 mm
- net /SCL: track 24.7 -> 25.4 mm
- added copper zone on B.Cu, net GNDA
- added copper zone on F.Cu, net GNDA
Other:
- board text added: "Jul 26"

Commit message: actually broke out dsdout whoops
Parts:
- J3, J4: footprint Connector_PinHeader_2.54mm:PinHeader_1x06_P2.54mm_Vertical -> Connector_PinHeader_2.54mm:PinHeader_1x07_P2.54mm_Vertical
- moved J4 2.54 mm to (144.2, 39.3)
- moved J3 2.52 mm to (162.1, 39.3)
- moved J1 2.31 mm to (154.6, 34.5)
Connections:
- IC1 pad 7: unconnected-(IC1-ASDOUT-Pad7) -> /ASDOUT
- J3 pad 1: /SCL -> /ASDOUT
- J3 pad 2: /SDA -> /SCL
- J3 pad 3: /I2C_DSDIN -> /SDA
- J3 pad 4: /I2C_SCLK -> /I2C_DSDIN
- J3 pad 5: /I2C_MCLK -> /I2C_SCLK
- J3 pad 6: /I2C_LRCK -> /I2C_MCLK
- J4 pad 1: /MIC_P -> unconnected-(J4-Pin_1-Pad1)
- J4 pad 2: /MIC_N -> /MIC_P
- J4 pad 3: /OUT_P -> /MIC_N
- J4 pad 4: /OUT_N -> /OUT_P
- J4 pad 5: +3V3 -> /OUT_N
- J4 pad 6: GND -> +3V3
Routing:
- net /ASDOUT: track 0.00 -> 32.6 mm, vias 0 -> 4
- net GNDA: track 74.9 -> 71.0 mm, vias 17 -> 16
- net /MIC_N: track 25.3 -> 27.4 mm
- net +3V3: track 32.1 -> 31.0 mm
- net /MIC_P: track 24.0 -> 24.9 mm
- net /I2C_DSDIN: track 14.7 -> 13.9 mm
- net /I2C_LRCK: track 15.8 -> 15.0 mm
Other:
- board size 21.4 x 34 mm -> 21.5 x 36.4 mm
- board text added: "ASDOUT"
